Commit message: urd5 file changes

File: src/assets/dishes/table_top.urdf (robot description, URDF)
Before this commit: robot table_top, 1 links, 0 joints
Links:
- link table_top_link: geometry collision box size=10 10 0.05; visual box size=10 10 0.05

File: ur_description/urdf/ur5e_left.urdf (robot description, URDF)
Before this commit: robot ur5e, 13 links, 12 joints
Joints:
- joint base_joint: origin xyz=0 0 0 rpy=0 0 0 -> xyz=-0.3 0 1 rpy=0 -90 0

File: ur_description/urdf/ur5e_right.urdf (robot description, URDF)
Before this commit: robot ur5e, 13 links, 12 joints
Joints:
- joint base_joint: origin xyz=0.6 0 0 rpy=0 0 0 -> xyz=0.3 0 1 rpy=0 90 0
