Commit message: initial scene definition

File: ur_description/urdf/ur5e_left.urdf (robot description, URDF)
Before this commit: robot ur5e, 13 links, 12 joints
Joints:
- joint base_joint: origin xyz=-0.3 0 1 rpy=0 -90 0 -> xyz=-0.17 0 1.27 rpy=0 -90 0

File: ur_description/urdf/ur5e_right.urdf (robot description, URDF)
Before this commit: robot ur5e, 13 links, 12 joints
Joints:
- joint base_joint: origin xyz=0.3 0 1 rpy=0 90 0 -> xyz=0.17 0 1.27 rpy=0 90 0
